File: debugger_base/debugger_base_ft4232h.kicad_sch (KiCad schematic)
At the start: 30 parts, among them SW1 RESET, X2 Channel A, X3 Channel B, X4 Channel C, X5 Channel D, Y1 12MHz

Commit message: decrease clearance of copper pours
Other:
- title: (none) -> FT4232 Debugger Base
