File: debugger_base/debugger_base_power.kicad_sch (KiCad schematic)
At the start: 15 parts, among them X1 USB-C Receptacle

Commit message: decrease clearance of copper pours
Other:
- title: (none) -> FT4232 Debugger Base
Changed lines of the file:
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@@
 	(generator_version "8.0")
 	(paper "A4")
+	(title_block
+		(title "FT4232 Debugger Base")
+		(date "2024-02-10")
+		(rev "v1.0")
+		(comment 4 "Simon Brenninger")
+	)
 	(junction
 		(at 90.17 57.15)
@@
 	(label "CONN_D-"
 		(at 72.39 72.39 0)
-		(fields_autoplaced yes)
 		(effects
 			(font
@@
 	(label "CONN_D+"
 		(at 72.39 74.93 0)
-		(fields_autoplaced yes)
 		(effects
 			(font
@@
 		(shape input)
 		(at 195.58 132.08 0)
-		(fields_autoplaced yes)
 		(effects
 			(font
@@
 		(shape input)
 		(at 139.7 59.69 0)
-		(fields_autoplaced yes)
 		(effects
 			(font
@@
 		(shape input)
 		(at 195.58 135.89 0)
-		(fields_autoplaced yes)
 		(effects
 			(font
@@
 		(shape input)
 		(at 195.58 128.27 0)
-		(fields_autoplaced yes)
 		(effects
 			(font
@@
 		(shape input)
 		(at 139.7 85.09 0)
-		(fields_autoplaced yes)
-		(effects
-			(font
+		(effects
+			(font
